File: PEP101-BJT/PEP101-BJT.kicad_sch (KiCad schematic)
At the start: 12 parts, among them J1 Screw_Terminal_01x02, J3 Conn_01x02_Pin, J4 Conn_01x02_Pin, J5 Conn_01x02_Pin, J6 Conn_01x02_Pin, Q2 MMBT5551L

Commit message: fix
Parts:
- J3, J4, J5, J6: footprint Connector_PinHeader_2.54mm:PinHeader_2x01_P2.54mm_Vertical -> PEP_library:PinHeader_2x01_P2.54mm_Vertical
Changed lines of the file:
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@@
 			)
 		)
-		(property "Footprint" "Connector_PinHeader_2.54mm:PinHeader_2x01_P2.54mm_Vertical"
+		(property "Footprint" "PEP_library:PinHeader_2x01_P2.54mm_Vertical"
 			(at 92.71 54.61 0)
 			(effects
@@
 			)
 		)
-		(property "Footprint" "Connector_PinHeader_2.54mm:PinHeader_2x01_P2.54mm_Vertical"
+		(property "Footprint" "PEP_library:PinHeader_2x01_P2.54mm_Vertical"
 			(at 22.86 82.55 0)
 			(effects
@@
 			)
 		)
-		(property "Footprint" "Connector_PinHeader_2.54mm:PinHeader_2x01_P2.54mm_Vertical"
+		(property "Footprint" "PEP_library:PinHeader_2x01_P2.54mm_Vertical"
 			(at 92.71 46.99 0)
 			(effects
@@
 			)
 		)
-		(property "Footprint" "Connector_PinHeader_2.54mm:PinHeader_2x01_P2.54mm_Vertical"
+		(property "Footprint" "PEP_library:PinHeader_2x01_P2.54mm_Vertical"
 			(at 22.86 90.17 0)
 			(effects
