File: PEP102-MOSFET/PEP102-MOSFET.kicad_sch (KiCad schematic)
At the start: 13 parts, among them J1 Screw_Terminal_01x02, J3 Conn_01x02_Pin, J4 Conn_01x02_Pin, J5 Conn_01x02_Pin, J6 Conn_01x02_Pin, Q19 2N7002

Commit message: fix
Parts:
- J3, J4, J5, J6: footprint Connector_PinHeader_2.54mm:PinHeader_2x01_P2.54mm_Vertical -> PEP_library:PinHeader_2x01_P2.54mm_Vertical
- renumbered D14 to D1, Q19 to Q1, R2 to R1
Changed lines of the file:
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@@
 			)
 		)
-		(property "Footprint" "Connector_PinHeader_2.54mm:PinHeader_2x01_P2.54mm_Vertical"
+		(property "Footprint" "PEP_library:PinHeader_2x01_P2.54mm_Vertical"
 			(at 106.68 52.07 0)
 			(effects
@@
 		(dnp no)
 		(fields_autoplaced yes)
-		(property "Reference" "D14"
+		(property "Reference" "D1"
 			(at 64.77 91.4399 90)
 			(effects
@@
 			(project "PEP102-MOSFET"
 				(path "/4bec5ddf-adbf-41fb-a069-c7630bb0044a"
-					(reference "D14")
+					(reference "D1")
 					(unit 1)
 				)
@@
 			)
 		)
-		(property "Footprint" "Connector_PinHeader_2.54mm:PinHeader_2x01_P2.54mm_Vertical"
+		(property "Footprint" "PEP_library:PinHeader_2x01_P2.54mm_Vertical"
 			(at 22.86 85.09 0)
 			(effects
@@
 			)
 		)
-		(property "Footprint" "Connector_PinHeader_2.54mm:PinHeader_2x01_P2.54mm_Vertical"
+		(property "Footprint" "PEP_library:PinHeader_2x01_P2.54mm_Vertical"
 			(at 106.68 44.45 0)
 			(effects
@@
 		(dnp no)
 		(fields_autoplaced yes)
-		(property "Reference" "R2"
+		(property "Reference" "R1"
 			(at 45.72 78.74 90)
 			(effects
@@
 			(project ""
 				(path "/4bec5ddf-adbf-41fb-a069-c7630bb0044a"
-					(reference "R2")
+					(reference "R1")
 					(unit 1)
 				)
@@
 			)
 		)
-		(property "Footprint" "Connector_PinHeader_2.54mm:PinHeader_2x01_P2.54mm_Vertical"
+		(property "Footprint" "PEP_library:PinHeader_2x01_P2.54mm_Vertical"
 			(at 22.86 92.71 0)
 			(effects
@@
 		(on_board yes)
 		(dnp no)
-		(property "Reference" "Q19"
+		(property "Reference" "Q1"
 			(at 101.6 83.8199 0)
 			(effects
@@
 			(project "PEP102-MOSFET"
 				(path "/4bec5ddf-adbf-41fb-a069-c7630bb0044a"
-					(reference "Q19")
-					(unit 1)
-				)
+					(reference "Q1")
+					(unit 1)
+				)
