File: PEP102-MOSFET/PEP102-MOSFET.kicad_pcb (KiCad board)
At the start: 2 copper layers, 45 x 45 mm, 19 parts, among them J1 Screw_Terminal_01x02, J3 Conn_01x02_Pin, J4 Conn_01x02_Pin, J5 Conn_01x02_Pin, J6 Conn_01x02_Pin, Q19 2N7002

Commit message: fix
Parts:
- added REF**: ele_petnica_logo, PEP_library:ele_petnica_logo, F.Cu at (122.2, 133.0)
- J3, J4, J5, J6: footprint Connector_PinHeader_2.54mm:PinHeader_2x01_P2.54mm_Vertical -> PEP_library:PinHeader_2x01_P2.54mm_Vertical
- renumbered D14 to D1, Q19 to Q1, R2 to R1
Routing:
- net Net-(Q1-G): track 12.8 -> 9.40 mm
Other:
- board text added: "V_{cc}"
- board text added: "V_{d}"
- board text added: "V_{g}"
- board text added: "d"
- board text added: "g"
- board text added: "s"
- board text removed: "Q2"

Commit message: fix 202
Parts:
- moved REF** 5.28 mm to (122.2, 138.3)
