File: PEP201-pojacavac_klase_A/PEP201-pojacavac_klase_A.kicad_sch (KiCad schematic)
At the start: 18 parts, among them J1 Screw_Terminal_01x02, J2 Conn_01x02_Pin, J3 Conn_01x02_Pin, J4 Conn_01x02_Pin, J5 Conn_01x02_Pin, Q1 MMBT2222A

Commit message: fix
Parts:
- J2, J3, J4, J5: footprint Connector_PinHeader_2.54mm:PinHeader_1x02_P2.54mm_Vertical -> PEP_library:PinHeader_2x01_P2.54mm_Vertical
Changed lines of the file:
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@@
 			)
 		)
-		(property "Footprint" "Connector_PinHeader_2.54mm:PinHeader_1x02_P2.54mm_Vertical"
+		(property "Footprint" "PEP_library:PinHeader_2x01_P2.54mm_Vertical"
 			(at 107.95 25.4 0)
 			(effects
@@
 			)
 		)
-		(property "Footprint" "Connector_PinHeader_2.54mm:PinHeader_1x02_P2.54mm_Vertical"
+		(property "Footprint" "PEP_library:PinHeader_2x01_P2.54mm_Vertical"
 			(at 161.29 25.4 0)
 			(effects
@@
 			)
 		)
-		(property "Footprint" "Connector_PinHeader_2.54mm:PinHeader_1x02_P2.54mm_Vertical"
+		(property "Footprint" "PEP_library:PinHeader_2x01_P2.54mm_Vertical"
 			(at 147.32 25.4 0)
 			(effects
@@
 			)
 		)
-		(property "Footprint" "Connector_PinHeader_2.54mm:PinHeader_1x02_P2.54mm_Vertical"
+		(property "Footprint" "PEP_library:PinHeader_2x01_P2.54mm_Vertical"
 			(at 93.98 25.4 0)
 			(effects
