File: PEP201-pojacavac_klase_A/PEP201-pojacavac_klase_A.kicad_pcb (KiCad board)
At the start: 2 copper layers, 45 x 45 mm, 28 parts, among them J1 Screw_Terminal_01x02, J2 Conn_01x02_Pin, J3 Conn_01x02_Pin, J4 Conn_01x02_Pin, J5 Conn_01x02_Pin, Q1 MMBT2222A

Commit message: fix
Parts:
- J2, J3, J4, J5: footprint Connector_PinHeader_2.54mm:PinHeader_1x02_P2.54mm_Vertical -> PEP_library:PinHeader_2x01_P2.54mm_Vertical
- moved REF** 8.70 mm to (122.2, 136.3)
- turned J2 to 90 degrees
- turned J3 to -90 degrees
- turned J4 to 90 degrees
- turned J5 to -90 degrees
Other:
- board text added: "b"
- board text added: "c"
- board text added: "e"
- board text removed: "+"
- board text removed: "-"
