File: PEP202-emitter_follower/PEP202-emitter_follower.kicad_sch (KiCad schematic)
At the start: 15 parts, among them J1 Screw_Terminal_01x02, J2 Conn_01x02_Pin, J3 Conn_01x02_Pin, J4 Conn_01x02_Pin, J5 Conn_01x02_Pin, Q1 NPN

Commit message: 202
Parts:
- added C1: 10u, Capacitor_SMD:C_1206_3216Metric_Pad1.33x1.80mm_HandSolder, symbol Device:C
- added J6, J7: Conn_01x02_Pin, Connector_PinHeader_2.54mm:PinHeader_1x02_P2.54mm_Vertical, symbol Connector:Conn_01x02_Pin
- C2, C3: footprint PEP_library:C_1206_3216Metric -> Capacitor_SMD:C_1206_3216Metric_Pad1.33x1.80mm_HandSolder
- Q1: value NPN -> 2N3904
- R1, R2, R3: footprint PEP_library:R_smd_1206 -> Resistor_SMD:R_1206_3216Metric_Pad1.30x1.75mm_HandSolder
Connections:
- net GND is gone; now on net 0: R2.2, R3.2
- net 0: now also C1.1
- net Input signal: now also J6.1 (Pin_1)
- net Output signal: now also J7.2 (Pin_2)
- net Vcc: now also C1.2
- net at C3.2, Q1.2 (B), R1.2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: now also J6.2 (Pin_2)
- net at C2.1, Q1.3 (E), R3.1: now also J7.1 (Pin_1)
Other:
- moved on the sheet: C2, C3, Q1, R1, R2, R3

Commit message: fix
Parts:
- removed Q1: 2N3904, Package_TO_SOT_SMD:SOT-23, symbol Simulation_SPICE:NPN
- added Q1: MMBT2222A, Package_TO_SOT_SMD:SOT-23, symbol Transistor_BJT:MMBT2222A
- J2, J3, J4, J5, J6, J7: footprint Connector_PinHeader_2.54mm:PinHeader_1x02_P2.54mm_Vertical -> PEP_library:PinHeader_2x01_P2.54mm_Vertical
Connections:
- net Vcc: now also Q1.3 (C)
- net at C3.2, J6.2 (Pin_2), R1.2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: now also Q1.1 (B)
- net at C2.1, J7.1 (Pin_1), R3.1: now also Q1.2 (E)
