File: PEP202-emitter_follower/PEP202-emitter_follower.kicad_pcb (KiCad board)
At the start: 2 copper layers, 45 x 45 mm, 15 parts, among them J1 Screw_Terminal_01x02, J2 Conn_01x02_Pin, J3 Conn_01x02_Pin, J4 Conn_01x02_Pin, J5 Conn_01x02_Pin, Q1 NPN

Commit message: 202
Parts:
- added C1: 10u, Capacitor_SMD:C_1206_3216Metric_Pad1.33x1.80mm_HandSolder, F.Cu at (122.2, 114.2)
- added J6: Conn_01x02_Pin, Connector_PinHeader_2.54mm:PinHeader_1x02_P2.54mm_Vertical, F.Cu at (112.3, 127.1)
- added J7: Conn_01x02_Pin, Connector_PinHeader_2.54mm:PinHeader_1x02_P2.54mm_Vertical, F.Cu at (130.3, 127.1)
- C2, C3: footprint PEP_library:C_1206_3216Metric -> Capacitor_SMD:C_1206_3216Metric_Pad1.33x1.80mm_HandSolder
- Q1: value NPN -> 2N3904
- R1, R2, R3: footprint PEP_library:R_smd_1206 -> Resistor_SMD:R_1206_3216Metric_Pad1.30x1.75mm_HandSolder
- moved Q1 5.06 mm to (124.9, 122.0)
- moved C2 5.05 mm to (131.2, 122.0)
- moved J1 3.75 mm to (122.2, 107.0)
- moved R3 3.52 mm to (126.0, 128.6)
- moved R2 2.90 mm to (120.0, 128.6)
- moved C3 1.30 mm to (113.5, 122.8)
- moved R1 0.90 mm to (120.0, 121.4)
Connections:
- R2 pad 2: GND -> 0
- R3 pad 2: GND -> 0
Routing:
- net GND: track 8.00 -> 0.00 mm
- net Output signal: track 8.04 -> 15.1 mm
- net Input signal: track 7.96 -> 14.8 mm
- net Net-(J7-Pin_1): track 7.63 -> 13.8 mm
- net Net-(J6-Pin_2): track 21.7 -> 17.8 mm
- net 0: track 0.00 -> 3.45 mm, vias 109 -> 112
- net Vcc: track 21.1 -> 19.8 mm
Other:
- board text added: "PEP 202"
- board text removed: "PEP 007"
- board text removed: "TestPoint"

Commit message: fix
Parts:
- added REF**: ele_petnica_logo, PEP_library:ele_petnica_logo, F.Cu at (122.4, 135.8)
- J2, J3, J4, J5, J6, J7: footprint Connector_PinHeader_2.54mm:PinHeader_1x02_P2.54mm_Vertical -> PEP_library:PinHeader_2x01_P2.54mm_Vertical
- Q1: value 2N3904 -> MMBT2222A
- moved Q1 0.14 mm to (125.0, 121.9), turned to 90 degrees
- turned J2 to 90 degrees
- turned J3 to -90 degrees
- turned J4 to 90 degrees
- turned J5 to -90 degrees
- turned J6 to 0 degrees
- turned J7 to 0 degrees
Connections:
- Q1 pad 1: Vcc -> Net-(J6-Pin_2)
- Q1 pad 2: Net-(J6-Pin_2) -> Net-(J7-Pin_1)
- Q1 pad 3: Net-(J7-Pin_1) -> Vcc
Routing:
- net Input signal: track 14.8 -> 17.4 mm
- net Output signal: track 15.1 -> 17.6 mm
- net Vcc: track 19.8 -> 20.5 mm
- net Net-(J6-Pin_2): track 17.8 -> 17.2 mm
Other:
- board text added: "V_{out}"
- board text added: "b"
- board text added: "c"
- board text added: "e"

Commit message: fix 202
Parts:
- added REF**: NPNsilk, PEP_library:NPNsilk, F.Cu at (124.1, 120.5)
- added REF**: R_silk_symbol, PEP_library:R_silk_symbol, F.Cu at (125.9, 128.6)
- added REF**: C_silk_symbol, PEP_library:C_silk_symbol, F.Cu at (113.5, 120.5)
- added REF**: R_silk_symbol, PEP_library:R_silk_symbol, F.Cu at (117.9, 114.0)
- added REF**: C_silk_symbol, PEP_library:C_silk_symbol, F.Cu at (131.2, 123.3)
- added REF**: C_silk_symbol, PEP_library:C_silk_symbol, F.Cu at (129.9, 113.4)
- added REF**: R_silk_symbol, PEP_library:R_silk_symbol, F.Cu at (117.9, 128.6)
Other:
- board text added: "V_{cc}"
