File: PEP203-pojacavac_klase_AB/PEP203-pojacavac_klase_AB.kicad_pcb (KiCad board)
At the start: 2 copper layers, 45 x 45 mm, 32 parts, among them J1 Screw_Terminal_01x02, J2 Conn_01x02_Pin, J3 Conn_01x02_Pin, J4 Conn_01x02_Pin, J5 Conn_01x02_Pin, J6 Conn_01x02_Pin, Q2 MMBT5551L, Q3 MMBT5401

Commit message: fix
Parts:
- J2, J3, J4, J5, J6: footprint Connector_PinHeader_2.54mm:PinHeader_1x02_P2.54mm_Vertical -> PEP_library:PinHeader_2x01_P2.54mm_Vertical
- turned J2 to 90 degrees
- turned J3 to -90 degrees
- turned J4 to 90 degrees
- turned J5 to -90 degrees
- turned J6 to -90 degrees
Other:
- board text added: "PEP 203"
- board text removed: "+"
- board text removed: "-"
- board text removed: "PEP 201"
